File: PCB-Test.kicad_pcb (KiCad board)
At the start: 4 copper layers, 60 x 60 mm, 29 parts, among them J1 PM25_CONNECTOR, J10 EN_CONNECTOR, J2 OZONE_CONNECTOR, J3 ADAFRUIT_SCD40_CONNECTOR, J4 ADAFRUIT_SHT4X_CONNECTOR, J5 PWR_OUT_1, J6 PWR_OUT_2, J7 PWR_IN, J8 I2C_CONNECTOR, J9 EXT_PM25_CONNECTOR, U1 TPS22917DBV, U2 TPS22917DBV, U3 TPS22917DBV, U4 TPS22917DBV, U5 MCP1702T-5002E/MB

Commit message: Add BOM
Parts:
- added D1: LED, LED_SMD:LED_0603_1608Metric, F.Cu at (163.0, 106.5)
- added JP1: Jumper_2_Open, Connector_PinHeader_2.54mm:PinHeader_1x02_P2.54mm_Vertical, F.Cu at (168.0, 105.3)
- added R1: 4.7kΩ, Resistor_SMD:R_0603_1608Metric, F.Cu at (163.0, 102.7)
- moved J9 12.9 mm to (154.2, 96.8)
- moved J10 4.28 mm to (161.8, 90.8)
- moved J8 3.47 mm to (175.5, 105.2)
- moved J5 2.39 mm to (187.8, 105.2), turned to -90 degrees
- moved J6 2.29 mm to (195.5, 105.2), turned to -90 degrees
Routing:
- net /SHT4X_EN: track 24.4 -> 53.1 mm, vias 1 -> 0
- net /PM25_EN: track 36.6 -> 52.3 mm
- net /SCL: track 119.1 -> 103.8 mm, vias 0 -> 2
- net /SDA: track 126.9 -> 117.1 mm, vias 1 -> 4
- net /PM25_RST: track 56.1 -> 64.0 mm, vias 1 -> 0
- net /PM25_TX: track 56.2 -> 63.1 mm, vias 1 -> 0
- net Net-(D1-A): track 0.00 -> 4.76 mm
- net VCC: track 45.2 -> 41.1 mm
- net Net-(D1-K): track 0.00 -> 3.79 mm
- net /OZONE_EN: track 37.6 -> 40.2 mm
- net /PM25_SET: track 64.7 -> 63.3 mm, vias 1 -> 0
- net /PM25_RX: track 63.3 -> 62.2 mm, vias 1 -> 0
- net /SCD40_EN: track 44.1 -> 43.1 mm, vias 2 -> 0
- net GND: track 40.2 -> 39.2 mm, vias 12 -> 11
Other:
- board text added: "5v"
- board text added: "COPYRIGHT 2025 UofT Network Research Lab VERSION 1.0"
- board text added: "En to MC"
- board text added: "GND"
- board text added: "LED JUMPER"
- board text added: "NC"
- board text added: "OZ"
- board text added: "PM"
- board text added: "PM25 Connector"
- board text added: "PM25 to MC"
- board text added: "RST"
- board text added: "RX"
- board text added: "SCD"
- board text added: "SCL"
- board text added: "SDA"
- board text added: "SET"
- board text added: "SHT"
- board text added: "TX"
- board text added: "VCC"

Commit message: Generate production files
Routing:
- net /SDA: track 117.1 -> 120.5 mm, vias 4 -> 3
- net /OZONE_EN: track 40.2 -> 39.7 mm
Changed lines of the file:
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@@
-	)
-	(segment
-		(start 159.26 91.25)
-		(end 159.26 90.75)
-		(width 0.3)
-		(layer "F.Cu")
-		(net 8)
 	)
 	(segment
@@
 	(segment
 		(start 186.75 71.5)
-		(end 195.25 63)
+		(end 192.58 65.67)
+		(width 0.3)
+		(layer "F.Cu")
+		(net 17)
+	)
+	(segment
+		(start 183.75 71.5)
+		(end 186.75 71.5)
+		(width 0.3)
+		(layer "F.Cu")
+		(net 17)
+	)
+	(segment
+		(start 192.58 65.67)
+		(end 192.58 55.75)
 		(width 0.3)
 		(layer "F.Cu")
@@
 		(start 168.5 71.5)
 		(end 178.75 71.5)
-		(width 0.3)
-		(layer "F.Cu")
-		(net 17)
-	)
-	(segment
-		(start 183.75 71.5)
-		(end 186.75 71.5)
 		(width 0.3)
 		(layer "F.Cu")
@@
 	)
 	(via
-		(at 195.25 63)
-		(size 0.7)
-		(drill 0.3)
-		(layers "F.Cu" "B.Cu")
-		(net 17)
-	)
-	(via
 		(at 178.75 71.5)
 		(size 0.7)
@@
 	)
 	(segment
-		(start 192.83 63)
-		(end 192.58 62.75)
-		(width 0.3)
-		(layer "B.Cu")
-		(net 17)
-	)
-	(segment
 		(start 192.5 66.75)
 		(end 192.5 66.25)
@@
 	)
 	(segment
-		(start 192.58 62.75)
+		(start 192.58 66.17)
 		(end 192.58 55.75)
 		(width 0.3)
@@
 	)
 	(segment
-		(start 195.25 63)
-		(end 192.83 63)
-		(width 0.3)
-		(layer "B.Cu")
-		(net 17)
-	)
-	(segment
 		(start 178.75 71.5)
 		(end 183.75 71.5)
-		(width 0.3)
-		(layer "B.Cu")
-		(net 17)
-	)
-	(segment
-		(start 192.58 66.17)
-		(end 192.58 62.75)
 		(width 0.3)
 		(layer "B.Cu")
@@
 	)
 	(segment
-		(start 194.475 101.7375)
+		(start 191.2875 101.7375)
 		(end 197.9625 101.7375)
 		(width 0.8)
@@
 		(width 0.8)
 		(layer "B.Cu")
-		(net 26)
-	)
-	(segment
-		(start 191.2875 101.7375)
-		(end 194.475 101.7375)
-		(width 0.8)
-		(layer "B.Cu")

Commit message: Finalize
Parts:
- moved J1 8.75 mm to (173.8, 56.2), turned to 180 degrees
- moved J9 7.50 mm to (161.8, 96.8), turned to -90 degrees
Routing:
- net /PM25_VCC: track 14.1 -> 21.2 mm
- net /PM25_SET: track 63.3 -> 67.7 mm
- net /PM25_RX: track 62.2 -> 65.8 mm
- net /PM25_RST: track 64.0 -> 62.0 mm
- net /PM25_TX: track 63.1 -> 63.9 mm
