File: PCB-Test.kicad_sch (KiCad schematic)
At the start: 29 parts, among them J1 PM25_CONNECTOR, J10 EN_CONNECTOR, J2 OZONE_CONNECTOR, J3 ADAFRUIT_SCD40_CONNECTOR, J4 ADAFRUIT_SHT4X_CONNECTOR, J5 PWR_OUT_1, J6 PWR_OUT_2, J7 PWR_IN, J8 I2C_CONNECTOR, J9 EXT_PM25_CONNECTOR, U1 TPS22917DBV, U2 TPS22917DBV, U3 TPS22917DBV, U4 TPS22917DBV, U5 MCP1702T-5002E/MB

Commit message: Add BOM
Parts:
- added D1: LED, LED_SMD:LED_0603_1608Metric, symbol Device:LED
- added JP1: Jumper_2_Open, Connector_PinHeader_2.54mm:PinHeader_1x02_P2.54mm_Vertical, symbol Jumper:Jumper_2_Open
- added R1: 4.7kΩ, Resistor_SMD:R_0603_1608Metric, symbol Device:R_US
- C1, C2, C3, C4, C5, C6, C7, C8: LCSC (none) -> C28323
- C10, C9: LCSC (none) -> C1779
- U1, U2, U3, U4: LCSC (none) -> C2680344
- U5: LCSC (none) -> C18299
Connections:
- net +5V: now also JP1.2 (B)
- net GND: now also R1.1
- new net: D1.1 (K), R1.2
- new net: D1.2 (A), JP1.1 (A)
Other:
- company: (none) -> UofT Network Research Lab
- title: (none) -> AQ Sensor Controll Board
- moved on the sheet: C10, C9, H1, H2, H3, H4, J10, J5, J6, J7, J8, J9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

Commit message: Generate production files
Parts:
- U1, U2, U3, U4: LCSC C2680344 -> C2681320
Changed lines of the file:
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@@
 			)
 		)
-		(property "LCSC" "C2680344"
+		(property "LCSC" "C2681320"
 			(at 50.8 38.1 0)
 			(effects
@@
 			)
 		)
-		(property "LCSC" "C2680344"
+		(property "LCSC" "C2681320"
 			(at 50.8 115.57 0)
 			(effects
@@
 			)
 		)
-		(property "LCSC" "C2680344"
+		(property "LCSC" "C2681320"
 			(at 50.8 90.17 0)
 			(effects
@@
 			)
 		)
-		(property "LCSC" "C2680344"
+		(property "LCSC" "C2681320"
 			(at 50.8 63.5 0)
 			(effects

Commit message: Finalize
Parts:
- J1: LCSC (none) -> C240845
Changed lines of the file:
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@@
 			)
 		)
-		(property "LCSC" ""
+		(property "LCSC" "C240845"
 			(at 134.62 38.1 0)
 			(effects
